File: hummingbird/hummingbird.kicad_pcb (KiCad board)
At the start: 4 copper layers, 53 x 20 mm, 47 parts, among them J1 USB_C_Receptacle_USB2.0_16P, J2 srv1, J3 srv2, J4 halleffect, J5 Conn_01x06, J6 Conn_01x02, J7 Conn_01x02, J8 PWR_IN, J9 Conn_02x02_Counter_Clockwise, Q1 AO3400A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

Commit message: completion, may have usbc placement bug
Parts:
- removed C20: 4u7, Capacitor_SMD:C_0402_1005Metric
- removed C21: 100n, Capacitor_SMD:C_0402_1005Metric
- removed U6: LPS22HH, Package_LGA:ST_HLGA-10_2x2mm_P0.5mm_LayoutBorder3x2y
- moved U5 22.7 mm to (172.2, 99.3), turned to -90 degrees
- moved C15 12.7 mm to (174.6, 100.3), turned to -90 degrees
- moved R1 11.9 mm to (174.6, 98.4), turned to -90 degrees
- moved R4 11.4 mm to (175.7, 98.4), turned to -90 degrees
- moved U3 3.73 mm to (165.5, 98.6)
- moved C10 3.69 mm to (167.8, 98.6)
- moved C11 3.68 mm to (165.5, 100.7)
- moved C12 3.65 mm to (168.8, 98.6)
- moved J1 0.30 mm to (158.7, 85.4)
Routing:
- net scl: track 21.5 -> 36.0 mm, vias 2 -> 4
- net sda: track 24.4 -> 38.2 mm
- net cs_pressure: track 12.5 -> 0.00 mm, vias 2 -> 0
- net sck: track 21.3 -> 12.2 mm, vias 4 -> 2
- net mosi: track 17.3 -> 10.3 mm
- net miso: track 14.8 -> 8.82 mm
- net int_imu: track 11.3 -> 6.96 mm
- net +3V3: track 23.8 -> 27.5 mm, vias 14 -> 17
- net cs_imu: track 16.7 -> 19.7 mm, vias 2 -> 0
- net GND: track 30.8 -> 28.3 mm, vias 33 -> 32

Commit message: Add STM32 skeleton code
Routing:
- net +3V3: track 27.5 -> 24.3 mm
Changed lines of the file:
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@@
 		)
 		(property "Value" "ICM-42688-P"
-			(at 0 2.2 360)
+			(at 0 2.2 0)
 			(layer "F.Fab")
 			(effects
@@
 		)
 		(fp_text user "${REFERENCE}"
-			(at 0 0 360)
+			(at 0 0 0)
 			(layer "F.Fab")
 			(effects
@@
 		)
 		(property "Value" "100n"
-			(at 0 1.16 360)
+			(at 0 1.16 0)
 			(layer "F.Fab")
 			(effects
@@
 		)
 		(fp_text user "${REFERENCE}"
-			(at 0 0 360)
+			(at 0 0 0)
 			(layer "F.Fab")
 			(effects
@@
 		(net 5)
 	)
-	(segment
-		(start 151.13 97.37)
-		(end 152.18 96.32)
-		(width 0.2)
-		(layer "B.Cu")
-		(net 5)
-	)
-	(segment
-		(start 149.34 97.37)
-		(end 151.13 97.37)
-		(width 0.2)
-		(layer "B.Cu")
-		(net 5)
-	)
